Commit message: feat(cameras): add D435i wrist/env cameras and MuJoCo test scene
Adds the D435i to the URDF (enable_cameras arg) and to the MJCF, raises the offscreen buffer to 1280x720, adds stacking cubes and a 'ready' initial keyframe. Camera publishing is configured by the CameraPlugin YAML in trossen_arm_moveit (auto_register_cameras=false).

File: urdf/wxai.urdf.xacro (robot description, xacro)
@@ -8,4 +8,13 @@
   <xacro:arg name="ip_address"                      default="192.168.1.2"/>
   <xacro:arg name="base_link_frame"                 default="base_link"/>
+  <!-- [cameras] block start -->
+  <!-- D435i wrist + environment cameras: same URDF for real hardware and MuJoCo -->
+  <xacro:arg name="enable_cameras"                  default="true"/>
+  <xacro:arg name="wrist_camera_xyz"                default="0.05 -0.03 0.06"/>
+  <xacro:arg name="wrist_camera_rpy"                default="0 0.785398163 0"/>
+  <xacro:arg name="env_camera_parent"               default="base_link"/>
+  <xacro:arg name="env_camera_xyz"                  default="0.2 0 1.0"/>
+  <xacro:arg name="env_camera_rpy"                  default="0 1.047197551 0"/>
+  <!-- [cameras] block end -->
   <xacro:if value="$(arg use_world_frame)">
     <link name="world"/>
@@ -19,4 +28,5 @@
   <xacro:include filename="$(find trossen_arm_description)/urdf/macros/_wxai.urdf.xacro" />
   <xacro:include filename="$(find trossen_arm_description)/urdf/macros/_common.urdf.xacro" />
+  <xacro:include filename="$(find trossen_arm_description)/urdf/peripherals/rs_d435i.urdf.xacro" />
   <xacro:trossen_black/>
   <xacro:wxai
@@ -26,3 +36,19 @@
     ros2_control_hardware_type="$(arg ros2_control_hardware_type)"
     ip_address="$(arg ip_address)"/>
+  <!-- [cameras] block start: instantiation below -->
+  <xacro:if value="$(arg enable_cameras)">
+    <xacro:sensor_d435i
+      name="wrist_camera"
+      parent="$(arg prefix)link_6"
+      use_nominal_extrinsics="true">
+      <origin xyz="$(arg wrist_camera_xyz)" rpy="$(arg wrist_camera_rpy)"/>
+    </xacro:sensor_d435i>
+    <xacro:sensor_d435i
+      name="env_camera"
+      parent="$(arg env_camera_parent)"
+      use_nominal_extrinsics="true">
+      <origin xyz="$(arg env_camera_xyz)" rpy="$(arg env_camera_rpy)"/>
+    </xacro:sensor_d435i>
+  </xacro:if> <!-- enable_cameras -->
+  <!-- [cameras] block end -->
 </robot>

File: urdf/wxai_mujoco.urdf.xacro (robot description, xacro)
@@ -7,4 +7,12 @@
       <plugin>mujoco_ros2_control/MujocoSystemInterface</plugin>
       <param name="mujoco_model">$(find trossen_arm_description)/urdf/mujoco/wxai_ros2_control_scene.xml</param>
+      <!-- Aplicada uma vez na inicialização; reset_world (sem "keyframe" na
+           request) volta para este mesmo estado, então o braço sempre
+           retorna à pose "ready" ao resetar o mundo. -->
+      <param name="initial_keyframe">ready</param>
+      <!-- Cameras are published by the CameraPlugin configured in
+           trossen_arm_moveit/config/mujoco_plugins.yaml. Disable the legacy auto-registration
+           so enable_cameras:=false really publishes no images. -->
+      <param name="auto_register_cameras">false</param>
     </hardware>
     <!-- Junta da Base -->
